File: jv-2080-enc.kicad_pcb (KiCad board)
At the start: 2 copper layers, 38 x 30 mm, 9 parts, among them J1 Conn_01x04, SW1 RotaryEncoder_Switch, U1 ATtiny13A-P

Commit message: Fixed miswired encoder connection. Added helpful silkscreen text. Bumped revision number from 0 to 1.
Connections:
- R1 pad 1: Net-(J1-Pad1) -> Net-(J1-Pad2)
- R2 pad 1: Net-(J1-Pad2) -> Net-(J1-Pad1)
Routing:
- net Net-(J1-Pad1): track 13.0 -> 11.7 mm
- net Net-(J1-Pad2): track 14.5 -> 15.6 mm
Other:
- board text added: "AND SOLDER J1 ON OPPOSITE SIDE"
- board text added: "HOMO ELECTRO- MAGNETICUS 2022"
- board text added: "INSTALL ENCODER ON THIS SIDE"
- board text added: "INSTALL J1 ON THIS SIDE"
- board text added: "PCB REV. 1"
- board text removed: "HOMO ELECTRO MAGNETICUS 2022"
- board text removed: "PCB REV. 0"
